File: hardware/pcb/kicad/zbox.kicad_pcb (KiCad board)
At the start: 2 copper layers, 58 x 64.5 mm, 24 parts, among them J1 USB_C_Receptacle_USB2.0_14P, J10 PAD_JBL, J11 PAD_LED_WS2812B, J12 PAD_JBL_PWR, J2 PAD_BAT_LIPO, J3 PAD_PN532_SPI, J7 PAD_BUTTONS, J8 ESP_LEFT, J9 ESP_RIGHT, Q1 BC547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

Commit message: doku
Other:
- board text added: "ZBox · v2.1 · 10/05/2026"
- board text removed: "Made with by Tata"
- board text removed: "ZBox · v2.0 · 13/04/2026"
Changed lines of the file:
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@@
 		(layer "Edge.Cuts")
 	)
-	(gr_text "ZBox · v2.0 · 13/04/2026"
+	(gr_text "ZBox · v2.1 · 10/05/2026"
 		(at 101.5 118.5 0)
 		(layer "F.SilkS")
@@
 			)
 			(justify left bottom)
-		)
-	)
-	(gr_text "Made with   by Tata"
-		(at 95 82.5 270)
-		(layer "F.SilkS")
-		(effects
-			(font
-				(size 1 1)
-				(thickness 0.2)
-				(bold yes)
-			)
-			(justify left bottom)
